File: KiCAD/GranulArduino v1.0/GranulArduino v1.0.sch (KiCad schematic (older format))
At the start: 51 parts, among them J1 GRAIN2_DECAY, J2 GRAIN1_FREQ, J3 GRAIN1_DECAY, J4 GRAIN2_FREQ, J5 SYNC, J6 OUTPUT, U4 TL074, U5 TL072, U6 ADS1115IDGS

Commit message: Renamed
Other:
- note added: "Arduino"
- note added: "Grain Controls"
- note added: "Output"
- note added: "Pitch Control"
Changed lines of the file:
@@
 NoConn ~ 6125 4700
 NoConn ~ 6125 4400
+Text Notes 675  7375 0    50   ~ 0
+Grain Controls
+Text Notes 5450 2475 0    50   ~ 0
+Pitch Control
+Text Notes 5450 5100 0    50   ~ 0
+Arduino
+Text Notes 5450 6400 0    50   ~ 0
+Output
 $EndSCHEMATC
